Commit message: update

File: urdf/navvis.xacro (robot description, xacro)
@@ -48,5 +48,5 @@
     <!-- Define the macro for the wheel link and joint !-->
     <xacro:macro name="xacro_name" params="side reflect">
-        <joint name="base_wheel_${side}_joint" type="fixed">
+        <joint name="base_wheel_${side}_joint" type="continuous">
             <parent link="base" />
             <child link="wheel_${side}" />
